Commit message: feat: migrate to Gazebo Fortress and standardize licenses
- Migrate simulation infrastructure to Gazebo Fortress (Ignition)
- Replace legacy launch files with unified bringup.launch.py
- Add warehouse.sdf world and update URDF/Xacro plugins
- Apply Apache-2.0 license headers to source files and add LICENSE
- Update package.xml manifests and CMakeLists.txt for linting compliance
- Fix build/test issues verified by local_ci.bash

File: src/mona_description/urdf/imu.xacro (robot description, xacro)
@@ -1,4 +1,17 @@
 <?xml version="1.0"?>
 <robot xmlns:xacro="http://www.ros.org/wiki/xacro">
+<!-- Copyright 2026 vladubase                                                   -->
+<!--                                                                            -->
+<!-- Licensed under the Apache License, Version 2.0 (the "License");            -->
+<!-- you may not use this file except in compliance with the License.           -->
+<!-- You may obtain a copy of the License at                                    -->
+<!--                                                                            -->
+<!--     http://www.apache.org/licenses/LICENSE-2.0                             -->
+<!--                                                                            -->
+<!-- Unless required by applicable law or agreed to in writing, software        -->
+<!-- distributed under the License is distributed on an "AS IS" BASIS,          -->
+<!-- WITHOUT WARRANTIES OR CONDITIONS OF ANY KIND, either express or implied.   -->
+<!-- See the License for the specific language governing permissions and        -->
+<!-- limitations under the License.                                             -->
     <xacro:macro name="imu_sensor" params="name parent *origin">
         <link name="${name}_link">
@@ -28,14 +41,21 @@
                 <always_on>true</always_on>
                 <update_rate>100</update_rate>
-                <visualize>true</visualize>
-                <topic>__default_topic__</topic>
-                <plugin filename="libgazebo_ros_imu_sensor.so" name="${name}_plugin">
-                    <ros>
-                        <remapping>~/out:=${name}/data</remapping>
-                    </ros>
-                    <initial_orientation_as_reference>false</initial_orientation_as_reference>
-                </plugin>
+                <visualize>false</visualize>
+                <topic>/${name}/data</topic>
                 <pose>0 0 0 0 0 0</pose>
-            </sensor>
+                <ignition_frame_id>${name}_link</ignition_frame_id>
+                <imu>
+                    <angular_velocity>
+                        <x><noise type="gaussian"><mean>0.0</mean><stddev>0.0</stddev></noise></x>
+                        <y><noise type="gaussian"><mean>0.0</mean><stddev>0.0</stddev></noise></y>
+                        <z><noise type="gaussian"><mean>0.0</mean><stddev>0.0</stddev></noise></z>
+                    </angular_velocity>
+                    <linear_acceleration>
+                        <x><noise type="gaussian"><mean>0.0</mean><stddev>0.0</stddev></noise></x>
+                        <y><noise type="gaussian"><mean>0.0</mean><stddev>0.0</stddev></noise></y>
+                        <z><noise type="gaussian"><mean>0.0</mean><stddev>0.0</stddev></noise></z>
+                    </linear_acceleration>
+                </imu>
+                </sensor>
         </gazebo>
     </xacro:macro>

File: src/mona_description/urdf/lidar.xacro (robot description, xacro)
@@ -1,13 +1,21 @@
 <?xml version="1.0"?>
 <robot xmlns:xacro="http://www.ros.org/wiki/xacro">
+<!-- Copyright 2026 vladubase                                                   -->
+<!--                                                                            -->
+<!-- Licensed under the Apache License, Version 2.0 (the "License");            -->
+<!-- you may not use this file except in compliance with the License.           -->
+<!-- You may obtain a copy of the License at                                    -->
+<!--                                                                            -->
+<!--     http://www.apache.org/licenses/LICENSE-2.0                             -->
+<!--                                                                            -->
+<!-- Unless required by applicable law or agreed to in writing, software        -->
+<!-- distributed under the License is distributed on an "AS IS" BASIS,          -->
+<!-- WITHOUT WARRANTIES OR CONDITIONS OF ANY KIND, either express or implied.   -->
+<!-- See the License for the specific language governing permissions and        -->
+<!-- limitations under the License.                                             -->
     <xacro:property name="lidar_radius" value="0.055"/>
     <xacro:property name="lidar_height" value="0.080"/>
     <xacro:property name="lidar_weight" value="0.070"/>
     <xacro:macro name="lidar_sensor" params="name parent *origin">
-        <joint name="${name}_joint" type="fixed">
-            <xacro:insert_block name="origin" />
-            <parent link="${parent}"/>
-            <child link="${name}_link"/>
-        </joint>
         <link name="${name}_link">
             <visual>
@@ -26,8 +34,16 @@
             </inertial>
         </link>
+        <joint name="${name}_joint" type="fixed">
+            <xacro:insert_block name="origin" />
+            <parent link="${parent}"/>
+            <child link="${name}_link"/>
+        </joint>
         <gazebo reference="${name}_link">
-            <sensor name="${name}" type="ray">
+            <sensor name="${name}" type="lidar">    <!-- or 'gpu_lidar' -->
+                <pose>0 0 0 0 0 0</pose>
+                <topic>${name}/scan</topic>
                 <always_on>true</always_on>
-                <visualize>true</visualize> <update_rate>15</update_rate>
+                <visualize>true</visualize>
+                <update_rate>10</update_rate>
                 <ray>
                     <scan>
@@ -50,13 +66,12 @@
                     </noise>
                 </ray>
-                <plugin name="${name}_controller" filename="libgazebo_ros_ray_sensor.so">
-                    <ros>
-                        <remapping>~/out:=${name}/scan</remapping>
-                    </ros>
-                    <output_type>sensor_msgs/LaserScan</output_type>
-                    <frame_name>${name}_link</frame_name>
-                </plugin>
-            </sensor>
-            <material>Gazebo/Yellow</material>
+                </sensor>
+            <visual>
+                <material>
+                    <ambient>1.0 0.8 0.0 1.0</ambient>
+                    <diffuse>1.0 0.8 0.0 1.0</diffuse>
+                    <specular>0.5 0.5 0.5 1.0</specular>
+                </material>
+            </visual>
         </gazebo>
     </xacro:macro>

File: src/mona_description/urdf/mona.urdf.xacro (robot description, xacro)
@@ -1,4 +1,19 @@
 <?xml version="1.0"?>
-<robot xmlns:xacro="http://www.ros.org/wiki/xacro" name="mona">
+<robot xmlns:xacro="http://www.ros.org/wiki/xacro"
+       xmlns:ignition="http://gazebosim.org/schema"
+       name="mona">
+<!-- Copyright 2026 vladubase                                                   -->
+<!--                                                                            -->
+<!-- Licensed under the Apache License, Version 2.0 (the "License");            -->
+<!-- you may not use this file except in compliance with the License.           -->
+<!-- You may obtain a copy of the License at                                    -->
+<!--                                                                            -->
+<!--     http://www.apache.org/licenses/LICENSE-2.0                             -->
+<!--                                                                            -->
+<!-- Unless required by applicable law or agreed to in writing, software        -->
+<!-- distributed under the License is distributed on an "AS IS" BASIS,          -->
+<!-- WITHOUT WARRANTIES OR CONDITIONS OF ANY KIND, either express or implied.   -->
+<!-- See the License for the specific language governing permissions and        -->
+<!-- limitations under the License.                                             -->
     <xacro:include filename="wheel.xacro"/>
     <xacro:include filename="lidar.xacro"/>
@@ -7,11 +22,14 @@
         <color rgba="1.0 0.5 0.0 1.0"/>
     </material>
+    <material name="white">
+        <color rgba="1.0 1.0 1.0 1.0"/>
+    </material>
     <xacro:property name="base_length"  value="1.25"/>
     <xacro:property name="base_width"   value="0.80"/>
     <xacro:property name="base_height"  value="0.30"/>
-    <xacro:property name="base_weight"  value="150.0"/>
+    <xacro:property name="base_weight"  value="200.0"/>
     <xacro:property name="robot_road_clearance" value="0.02"/>
-    <xacro:property name="wheel_base_x" value="${0.8 / 2}"/>
-    <xacro:property name="wheel_base_y" value="${base_width/2   - wheel_width/2}"/>
+    <xacro:property name="wheel_base_x" value="0.8"/>
+    <xacro:property name="wheel_base_y" value="${base_width - wheel_width}"/>
     <xacro:property name="wheel_base_z" value="${-base_height/2 - robot_road_clearance + wheel_radius}"/>
     <xacro:property name="lidar_offset_x" value="${base_length/2 - 0.06}"/>
@@ -20,5 +38,5 @@
     <xacro:property name="robot_spawn_x" value="0.0"/>
     <xacro:property name="robot_spawn_y" value="0.0"/>
-    <xacro:property name="robot_spawn_z" value="${(robot_road_clearance+0.003) + (base_height/2)}"/>
+    <xacro:property name="robot_spawn_z" value="${(robot_road_clearance) + (base_height/2)}"/>
     <!-- BASE FOOTPRINT -->
     <link name="base_footprint"/>
@@ -51,16 +69,22 @@
     </link>
     <gazebo reference="base_link">
-        <material>Gazebo/Orange</material>
+        <visual>
+            <material>
+                <ambient>1.0 0.25 0.0 1.0</ambient>
+                <diffuse>1.0 0.25 0.0 1.0</diffuse>
+                <specular>0.2 0.2 0.2 1.0</specular>
+            </material>
+        </visual>
     </gazebo>
     <!-- WHEELS -->
-    <xacro:mecanum_wheel name="wheel_front_left"  x="${wheel_base_x}"  y="${wheel_base_y}"  flip_visual="1"  parent="base_link" height_offset="${wheel_base_z}"/>
-    <xacro:mecanum_wheel name="wheel_rear_left"   x="-${wheel_base_x}" y="${wheel_base_y}"  flip_visual="1"  parent="base_link" height_offset="${wheel_base_z}"/>
-    <xacro:mecanum_wheel name="wheel_front_right" x="${wheel_base_x}"  y="-${wheel_base_y}" flip_visual="-1" parent="base_link" height_offset="${wheel_base_z}"/>
-    <xacro:mecanum_wheel name="wheel_rear_right"  x="-${wheel_base_x}" y="-${wheel_base_y}" flip_visual="-1" parent="base_link" height_offset="${wheel_base_z}"/>
+    <xacro:mecanum_wheel name="wheel_front_left"  x="${wheel_base_x/2}"  y="${wheel_base_y/2}"  sx="1"  sy="1"  parent="base_link" height_offset="${wheel_base_z}" fdir="1 1 0"/>
+    <xacro:mecanum_wheel name="wheel_front_right" x="${wheel_base_x/2}"  y="-${wheel_base_y/2}" sx="1"  sy="-1" parent="base_link" height_offset="${wheel_base_z}" fdir="1 -1 0"/>
+    <xacro:mecanum_wheel name="wheel_back_left"   x="-${wheel_base_x/2}" y="${wheel_base_y/2}"  sx="-1" sy="1"  parent="base_link" height_offset="${wheel_base_z}" fdir="1 -1 0"/>
+    <xacro:mecanum_wheel name="wheel_back_right"  x="-${wheel_base_x/2}" y="-${wheel_base_y/2}" sx="-1" sy="-1" parent="base_link" height_offset="${wheel_base_z}" fdir="1 1 0"/>
     <!-- LIDARS -->
     <xacro:lidar_sensor name="lidar_front" parent="base_link">
         <origin xyz="${lidar_offset_x} 0 ${lidar_offset_z}" rpy="0 0 0"/>
     </xacro:lidar_sensor>
-    <xacro:lidar_sensor name="lidar_rear" parent="base_link">
+    <xacro:lidar_sensor name="lidar_back" parent="base_link">
         <origin xyz="-${lidar_offset_x} 0 ${lidar_offset_z}" rpy="0 0 ${pi}"/>
     </xacro:lidar_sensor>
@@ -93,29 +117,47 @@
     </joint>
     <gazebo reference="led_strip_link">
-        <material>Gazebo/WhiteGlow</material>
+        <visual>
+            <material>
+                <ambient>1 1 1 1</ambient>
+                <diffuse>1 1 1 1</diffuse>
+                <specular>1 1 1 1</specular>
+                <emissive>1.0 1.0 1.0 1.0</emissive>
+            </material>
+        </visual>
     </gazebo>
     <!-- PLUGIN CONNECTIONS -->
     <gazebo>
-        <plugin name="object_controller" filename="libgazebo_ros_planar_move.so">
-            <ros>
-                <remapping>odom:=odom/unfiltered</remapping>
-            </ros>
-            <command_topic>cmd_vel</command_topic>
-            <odometry_topic>odom</odometry_topic>
-            <odometry_frame>odom</odometry_frame>
-            <odometry_rate>20.0</odometry_rate>
-            <robot_base_frame>base_footprint</robot_base_frame>
-            <publish_odom>true</publish_odom>
-            <publish_odom_tf>true</publish_odom_tf>
+        <!-- TF -->
+        <plugin filename="libignition-gazebo-joint-state-publisher-system.so"
+                name="ignition::gazebo::systems::JointStatePublisher">
+            <topic>joint_states</topic>
         </plugin>
-        <plugin name="joint_state_publisher" filename="libgazebo_ros_joint_state_publisher.so">
-            <ros>
-                <remapping>~/out:=joint_states</remapping>
-            </ros>
-            <update_rate>30</update_rate>
-            <joint_name>wheel_front_left_joint</joint_name>
-            <joint_name>wheel_front_right_joint</joint_name>
-            <joint_name>wheel_rear_left_joint</joint_name>
-            <joint_name>wheel_rear_right_joint</joint_name>
+        <!-- Mecanum Wheels -->
+        <plugin filename="libignition-gazebo-mecanum-drive-system.so"
+                name="ignition::gazebo::systems::MecanumDrive">
+            <front_left_joint>wheel_front_left_joint</front_left_joint>
+            <front_right_joint>wheel_front_right_joint</front_right_joint>
+            <back_left_joint>wheel_back_left_joint</back_left_joint>
+            <back_right_joint>wheel_back_right_joint</back_right_joint>
+            <wheel_separation>${wheel_base_y}</wheel_separation>
+            <wheelbase>${wheel_base_x}</wheelbase>
+            <wheel_radius>${wheel_radius}</wheel_radius>
+            <min_acceleration>-15.0</min_acceleration>
+            <max_acceleration>15.0</max_acceleration>
+            <topic>/cmd_vel</topic>
+            <odom_topic>/odom</odom_topic>
+            <tf_topic>/tf</tf_topic>
+            <frame_id>odom</frame_id>
+            <child_frame_id>base_footprint</child_frame_id>
+            <odom_publish_frequency>50</odom_publish_frequency>
+        </plugin>
+        <!-- Sensor: IMU -->
+        <plugin filename="libignition-gazebo-imu-system.so"
+                name="ignition::gazebo::systems::Imu">
+        </plugin>
+        <!-- Sensor: LiDAR -->
+        <plugin filename="libignition-gazebo-sensors-system.so"
+                name="ignition::gazebo::systems::Sensors">
+            <render_engine>ogre2</render_engine>
         </plugin>
     </gazebo>

File: src/mona_description/urdf/wheel.xacro (robot description, xacro)
@@ -1,13 +1,28 @@
 <?xml version="1.0"?>
-<robot xmlns:xacro="http://www.ros.org/wiki/xacro">
+<robot xmlns:xacro="http://www.ros.org/wiki/xacro"
+       xmlns:ignition="http://gazebosim.org/schema">
+<!-- Copyright 2026 vladubase                                                   -->
+<!--                                                                            -->
+<!-- Licensed under the Apache License, Version 2.0 (the "License");            -->
+<!-- you may not use this file except in compliance with the License.           -->
+<!-- You may obtain a copy of the License at                                    -->
+<!--                                                                            -->
+<!--     http://www.apache.org/licenses/LICENSE-2.0                             -->
+<!--                                                                            -->
+<!-- Unless required by applicable law or agreed to in writing, software        -->
+<!-- distributed under the License is distributed on an "AS IS" BASIS,          -->
+<!-- WITHOUT WARRANTIES OR CONDITIONS OF ANY KIND, either express or implied.   -->
+<!-- See the License for the specific language governing permissions and        -->
+<!-- limitations under the License.                                             -->
     <xacro:property name="wheel_radius" value="0.127"/>
     <xacro:property name="wheel_width"  value="0.132"/>
-    <xacro:property name="wheel_weight" value="15.0"/>
-    <xacro:macro name="mecanum_wheel" params="name x y flip_visual parent height_offset">
+    <xacro:property name="wheel_weight" value="10.0"/>
+    <xacro:macro name="mecanum_wheel" params="name x y sx sy parent height_offset fdir">
         <link name="${name}_link">
             <visual>
                 <origin xyz="0 0 0" rpy="${pi/2} 0 0"/>
                 <geometry>
-                    <mesh filename="package://mona_description/meshes/wheels/mecanum_wheel.stl" scale="0.001 0.001 0.001"/>
+                    <mesh filename="package://mona_description/meshes/wheels/mecanum_wheel.stl"
+                          scale="${0.001 * sx} ${0.001 * sy} 0.001"/>
                 </geometry>
                 <material name="black">
@@ -18,5 +33,5 @@
                 <origin xyz="0 0 0" rpy="${pi/2} 0 0"/>
                 <geometry>
-                    <cylinder radius="${wheel_radius}" length="${wheel_width}"/>
+                    <sphere radius="${wheel_radius}"/>
                 </geometry>
             </collision>
@@ -34,9 +49,37 @@
             <origin xyz="${x} ${y} ${height_offset}" rpy="0 0 0"/>
             <axis xyz="0 1 0"/>
+            <!-- Damping (Н·м·с/рад): создаёт сопротивление, пропорциональное скорости.
+            Это предотвратит «бесконечное» вращение колес по инерции.-->
+            <!-- Friction (Н·м): минимальное усилие, нужное для начала вращения.
+            Помогает робоу удерживаться на месте и не «дрейфовать» от вибраций.-->
+            <limit effort="1000.0" velocity="20.0"/>
+            <dynamics damping="1.5" friction="1.0"/>
         </joint>
         <gazebo reference="${name}_link">
-            <material>Gazebo/Grey</material>
-            <mu1>0.8</mu1>
-            <mu2>0.8</mu2>
+            <visual>
+                <material>
+                    <ambient>0.1 0.1 0.1 1.0</ambient>
+                    <diffuse>0.1 0.1 0.1 1.0</diffuse>
+                    <specular>0.5 0.5 0.5 1.0</specular>
+                </material>
+            </visual>
+            <collision>
+                <surface>
+                    <friction>
+                        <ode>
+                            <fdir1 ignition:expressed_in="base_footprint">${fdir}</fdir1>   <!-- Ось роликов        -->
+                            <mu>0.05</mu>   <!-- Коэффициент трения вдоль оси fdir  (должен быть 0, чтобы катилось).-->
+                            <mu2>1.0</mu2>  <!-- Коэффициент трения поперёк оси fdir(должен быть 1, чтобы катилось).-->
+                        </ode>
+                    </friction>
+                    <contact>
+                        <ode>
+                            <kp>1e8</kp>
+                            <kd>10.0</kd>
+                            <min_depth>0.001</min_depth>
+                        </ode>
+                    </contact>
+                </surface>
+            </collision>
         </gazebo>
     </xacro:macro>
