Commit message: feat: Add lidar fusion and warehouse, remove mona_core
- Feat: Added 'mona_perception' for merging 4 LiDARs.
- Feat: Updated 'warehouse.sdf' with shelving and friction.
- Chore: Removed 'mona_core' (deprecated).
- CI: Added XML/Docker linting to local_ci.bash.
- Style: Updated license headers to SPDX format.
- Config: Added .clang-tidy configuration.

File: src/mona_description/urdf/imu.xacro (robot description, xacro)
@@ -1,62 +1,90 @@
-<?xml version="1.0"?>
+<?xml version="1.0" ?>
 <robot xmlns:xacro="http://www.ros.org/wiki/xacro">
-<!-- Copyright 2026 vladubase                                                   -->
-<!--                                                                            -->
-<!-- Licensed under the Apache License, Version 2.0 (the "License");            -->
-<!-- you may not use this file except in compliance with the License.           -->
-<!-- You may obtain a copy of the License at                                    -->
-<!--                                                                            -->
-<!--     http://www.apache.org/licenses/LICENSE-2.0                             -->
-<!--                                                                            -->
-<!-- Unless required by applicable law or agreed to in writing, software        -->
-<!-- distributed under the License is distributed on an "AS IS" BASIS,          -->
-<!-- WITHOUT WARRANTIES OR CONDITIONS OF ANY KIND, either express or implied.   -->
-<!-- See the License for the specific language governing permissions and        -->
-<!-- limitations under the License.                                             -->
-    <xacro:macro name="imu_sensor" params="name parent *origin">
-        <link name="${name}_link">
-            <visual>
-                <geometry>
-                    <box size="0.05 0.05 0.05"/>
-                </geometry>
-                <material name="red">
-                    <color rgba="1.0 0.0 0.0 1.0"/>
-                </material>
-            </visual>
-            <inertial>
-                <mass value="0.10"/>
-                <inertia ixx="0.00001" ixy="0" ixz="0"
-                         iyy="0.00001" iyz="0"
-                         izz="0.00001"/>
-            </inertial>
-        </link>
-        <joint name="${name}_joint" type="fixed">
-            <parent link="${parent}"/>
-            <child link="${name}_link"/>
-            <xacro:insert_block name="origin"/>
-        </joint>
-        <gazebo reference="${name}_link">
-            <gravity>true</gravity>
-            <sensor name="${name}_sensor" type="imu">
-                <always_on>true</always_on>
-                <update_rate>100</update_rate>
-                <visualize>false</visualize>
-                <topic>/${name}/data</topic>
-                <pose>0 0 0 0 0 0</pose>
-                <ignition_frame_id>${name}_link</ignition_frame_id>
-                <imu>
-                    <angular_velocity>
-                        <x><noise type="gaussian"><mean>0.0</mean><stddev>0.0</stddev></noise></x>
-                        <y><noise type="gaussian"><mean>0.0</mean><stddev>0.0</stddev></noise></y>
-                        <z><noise type="gaussian"><mean>0.0</mean><stddev>0.0</stddev></noise></z>
-                    </angular_velocity>
-                    <linear_acceleration>
-                        <x><noise type="gaussian"><mean>0.0</mean><stddev>0.0</stddev></noise></x>
-                        <y><noise type="gaussian"><mean>0.0</mean><stddev>0.0</stddev></noise></y>
-                        <z><noise type="gaussian"><mean>0.0</mean><stddev>0.0</stddev></noise></z>
-                    </linear_acceleration>
-                </imu>
-                </sensor>
-        </gazebo>
-    </xacro:macro>
+  <!-- Copyright 2026 vladubase                                                 -->
+  <!--                                                                          -->
+  <!-- Licensed under the Apache License, Version 2.0 (the "License");          -->
+  <!-- you may not use this file except in compliance with the License.         -->
+  <!-- You may obtain a copy of the License at                                  -->
+  <!--                                                                          -->
+  <!-- http://www.apache.org/licenses/LICENSE-2.0                               -->
+  <!--                                                                          -->
+  <!-- Unless required by applicable law or agreed to in writing, software      -->
+  <!-- distributed under the License is distributed on an "AS IS" BASIS,        -->
+  <!-- WITHOUT WARRANTIES OR CONDITIONS OF ANY KIND, either express or implied. -->
+  <!-- See the License for the specific language governing permissions and      -->
+  <!-- limitations under the License.                                           -->
+  <xacro:macro name="imu_sensor" params="name parent *origin">
+    <link name="${name}_link">
+      <visual>
+        <geometry>
+          <box size="0.05 0.05 0.05"/>
+        </geometry>
+        <material name="red">
+          <color rgba="1.0 0.0 0.0 1.0"/>
+        </material>
+      </visual>
+      <inertial>
+        <mass value="0.10"/>
+        <inertia ixx="0.00001" ixy="0" ixz="0" iyy="0.00001" iyz="0" izz="0.00001"/>
+      </inertial>
+    </link>
+    <joint name="${name}_joint" type="fixed">
+      <parent link="${parent}"/>
+      <child link="${name}_link"/>
+      <xacro:insert_block name="origin"/>
+    </joint>
+    <gazebo reference="${name}_link">
+      <gravity>true</gravity>
+      <sensor name="${name}_sensor" type="imu">
+        <always_on>true</always_on>
+        <update_rate>100</update_rate>
+        <visualize>false</visualize>
+        <topic>/${name}/data</topic>
+        <pose>0 0 0 0 0 0</pose>
+        <ignition_frame_id>${name}_link</ignition_frame_id>
+        <imu>
+          <angular_velocity>
+            <x>
+              <noise type="gaussian">
+                <mean>0.0</mean>
+                <stddev>0.0</stddev>
+              </noise>
+            </x>
+            <y>
+              <noise type="gaussian">
+                <mean>0.0</mean>
+                <stddev>0.0</stddev>
+              </noise>
+            </y>
+            <z>
+              <noise type="gaussian">
+                <mean>0.0</mean>
+                <stddev>0.0</stddev>
+              </noise>
+            </z>
+          </angular_velocity>
+          <linear_acceleration>
+            <x>
+              <noise type="gaussian">
+                <mean>0.0</mean>
+                <stddev>0.0</stddev>
+              </noise>
+            </x>
+            <y>
+              <noise type="gaussian">
+                <mean>0.0</mean>
+                <stddev>0.0</stddev>
+              </noise>
+            </y>
+            <z>
+              <noise type="gaussian">
+                <mean>0.0</mean>
+                <stddev>0.0</stddev>
+              </noise>
+            </z>
+          </linear_acceleration>
+        </imu>
+      </sensor>
+    </gazebo>
+  </xacro:macro>
 </robot>

File: src/mona_description/urdf/lidar.xacro (robot description, xacro)
@@ -1,78 +1,78 @@
-<?xml version="1.0"?>
+<?xml version="1.0" ?>
 <robot xmlns:xacro="http://www.ros.org/wiki/xacro">
-<!-- Copyright 2026 vladubase                                                   -->
-<!--                                                                            -->
-<!-- Licensed under the Apache License, Version 2.0 (the "License");            -->
-<!-- you may not use this file except in compliance with the License.           -->
-<!-- You may obtain a copy of the License at                                    -->
-<!--                                                                            -->
-<!--     http://www.apache.org/licenses/LICENSE-2.0                             -->
-<!--                                                                            -->
-<!-- Unless required by applicable law or agreed to in writing, software        -->
-<!-- distributed under the License is distributed on an "AS IS" BASIS,          -->
-<!-- WITHOUT WARRANTIES OR CONDITIONS OF ANY KIND, either express or implied.   -->
-<!-- See the License for the specific language governing permissions and        -->
-<!-- limitations under the License.                                             -->
-    <xacro:property name="lidar_radius" value="0.055"/>
-    <xacro:property name="lidar_height" value="0.080"/>
-    <xacro:property name="lidar_weight" value="0.070"/>
-    <xacro:macro name="lidar_sensor" params="name parent *origin">
-        <link name="${name}_link">
-            <visual>
-                <geometry>
-                    <cylinder radius="${lidar_radius}" length="${lidar_height}"/>
-                </geometry>
-                <material name="yellow">
-                    <color rgba="1.0 0.8 0.0 1.0"/>
-                </material>
-            </visual>
-            <inertial>
-                <mass value="${lidar_weight}"/>
-                <inertia ixx="${1.0/12.0 * lidar_weight * (3 * lidar_radius*lidar_radius + lidar_height*lidar_height)}" ixy="0" ixz="0"
-                         iyy="${1.0/12.0 * lidar_weight * (3 * lidar_radius*lidar_radius + lidar_height*lidar_height)}" iyz="0"
-                         izz="${1.0/2.0  * lidar_weight * lidar_radius*lidar_radius}"/>
-            </inertial>
-        </link>
-        <joint name="${name}_joint" type="fixed">
-            <xacro:insert_block name="origin" />
-            <parent link="${parent}"/>
-            <child link="${name}_link"/>
-        </joint>
-        <gazebo reference="${name}_link">
-            <sensor name="${name}" type="lidar">    <!-- or 'gpu_lidar' -->
-                <pose>0 0 0 0 0 0</pose>
-                <topic>${name}/scan</topic>
-                <always_on>true</always_on>
-                <visualize>true</visualize>
-                <update_rate>10</update_rate>
-                <ray>
-                    <scan>
-                        <horizontal>
-                            <samples>300</samples>
-                            <resolution>1</resolution>
-                            <min_angle>${-pi/2.4}</min_angle>
-                            <max_angle>${pi/2.4}</max_angle>
-                        </horizontal>
-                    </scan>
-                    <range>
-                        <min>0.10</min>
-                        <max>20.0</max>
-                        <resolution>0.01</resolution>
-                    </range>
-                    <noise>
-                        <type>gaussian</type>
-                        <mean>0.0</mean>
-                        <stddev>0.01</stddev>
-                    </noise>
-                </ray>
-                </sensor>
-            <visual>
-                <material>
-                    <ambient>1.0 0.8 0.0 1.0</ambient>
-                    <diffuse>1.0 0.8 0.0 1.0</diffuse>
-                    <specular>0.5 0.5 0.5 1.0</specular>
-                </material>
-            </visual>
-        </gazebo>
-    </xacro:macro>
+  <!-- Copyright 2026 vladubase                                                 -->
+  <!--                                                                          -->
+  <!-- Licensed under the Apache License, Version 2.0 (the "License");          -->
+  <!-- you may not use this file except in compliance with the License.         -->
+  <!-- You may obtain a copy of the License at                                  -->
+  <!--                                                                          -->
+  <!-- http://www.apache.org/licenses/LICENSE-2.0                               -->
+  <!--                                                                          -->
+  <!-- Unless required by applicable law or agreed to in writing, software      -->
+  <!-- distributed under the License is distributed on an "AS IS" BASIS,        -->
+  <!-- WITHOUT WARRANTIES OR CONDITIONS OF ANY KIND, either express or implied. -->
+  <!-- See the License for the specific language governing permissions and      -->
+  <!-- limitations under the License.                                           -->
+  <xacro:property name="lidar_radius" value="0.055"/>
+  <xacro:property name="lidar_height" value="0.080"/>
+  <xacro:property name="lidar_weight" value="0.070"/>
+  <xacro:macro name="lidar_sensor" params="name parent *origin">
+    <link name="${name}_link">
+      <visual>
+        <geometry>
+          <cylinder radius="${lidar_radius}" length="${lidar_height}"/>
+        </geometry>
+        <material name="yellow">
+          <color rgba="1.0 0.8 0.0 1.0"/>
+        </material>
+      </visual>
+      <inertial>
+        <mass value="${lidar_weight}"/>
+        <inertia ixx="${1.0/12.0 * lidar_weight * (3 * lidar_radius*lidar_radius + lidar_height*lidar_height)}" ixy="0" ixz="0" iyy="${1.0/12.0 * lidar_weight * (3 * lidar_radius*lidar_radius + lidar_height*lidar_height)}" iyz="0" izz="${1.0/2.0 * lidar_weight * lidar_radius*lidar_radius}"/>
+      </inertial>
+    </link>
+    <joint name="${name}_joint" type="fixed">
+      <xacro:insert_block name="origin"/>
+      <parent link="${parent}"/>
+      <child link="${name}_link"/>
+    </joint>
+    <gazebo reference="${name}_link">
+      <sensor name="${name}" type="gpu_lidar">  <!-- or 'lidar' -->
+        <pose>0 0 0 0 0 0</pose>
+        <topic>${name}/scan</topic>
+        <always_on>true</always_on>
+        <visualize>true</visualize>
+        <update_rate>10</update_rate>
+        <gz_frame_id>${name}_link</gz_frame_id>
+        <ign_frame_id>${name}_link</ign_frame_id>
+        <ray>
+          <scan>
+            <horizontal>
+              <samples>300</samples>
+              <resolution>1</resolution>
+              <min_angle>${-pi/2.4}</min_angle>
+              <max_angle>${pi/2.4}</max_angle>
+            </horizontal>
+          </scan>
+          <range>
+            <min>0.10</min>
+            <max>20.0</max>
+            <resolution>0.01</resolution>
+          </range>
+          <noise>
+            <type>gaussian</type>
+            <mean>0.0</mean>
+            <stddev>0.01</stddev>
+          </noise>
+        </ray>
+      </sensor>
+      <visual>
+        <material>
+          <ambient>1.0 0.8 0.0 1.0</ambient>
+          <diffuse>1.0 0.8 0.0 1.0</diffuse>
+          <specular>0.5 0.5 0.5 1.0</specular>
+        </material>
+      </visual>
+    </gazebo>
+  </xacro:macro>
 </robot>
