Commit message: feat: Add lidar fusion and warehouse, remove mona_core
- Feat: Added 'mona_perception' for merging 4 LiDARs.
- Feat: Updated 'warehouse.sdf' with shelving and friction.
- Chore: Removed 'mona_core' (deprecated).
- CI: Added XML/Docker linting to local_ci.bash.
- Style: Updated license headers to SPDX format.
- Config: Added .clang-tidy configuration.

File: src/mona_description/urdf/wheel.xacro (robot description, xacro)
@@ -1,86 +1,72 @@
-<?xml version="1.0"?>
+<?xml version="1.0" ?>
 <robot xmlns:xacro="http://www.ros.org/wiki/xacro"
        xmlns:ignition="http://gazebosim.org/schema">
-<!-- Copyright 2026 vladubase                                                   -->
-<!--                                                                            -->
-<!-- Licensed under the Apache License, Version 2.0 (the "License");            -->
-<!-- you may not use this file except in compliance with the License.           -->
-<!-- You may obtain a copy of the License at                                    -->
-<!--                                                                            -->
-<!--     http://www.apache.org/licenses/LICENSE-2.0                             -->
-<!--                                                                            -->
-<!-- Unless required by applicable law or agreed to in writing, software        -->
-<!-- distributed under the License is distributed on an "AS IS" BASIS,          -->
-<!-- WITHOUT WARRANTIES OR CONDITIONS OF ANY KIND, either express or implied.   -->
-<!-- See the License for the specific language governing permissions and        -->
-<!-- limitations under the License.                                             -->
-    <xacro:property name="wheel_radius" value="0.127"/>
-    <xacro:property name="wheel_width"  value="0.132"/>
-    <xacro:property name="wheel_weight" value="10.0"/>
-    <xacro:macro name="mecanum_wheel" params="name x y sx sy parent height_offset fdir">
-        <link name="${name}_link">
-            <visual>
-                <origin xyz="0 0 0" rpy="${pi/2} 0 0"/>
-                <geometry>
-                    <mesh filename="package://mona_description/meshes/wheels/mecanum_wheel.stl"
-                          scale="${0.001 * sx} ${0.001 * sy} 0.001"/>
-                </geometry>
-                <material name="black">
-                    <color rgba="0.1 0.1 0.1 1.0"/>
-                </material>
-            </visual>
-            <collision>
-                <origin xyz="0 0 0" rpy="${pi/2} 0 0"/>
-                <geometry>
-                    <sphere radius="${wheel_radius}"/>
-                </geometry>
-            </collision>
-            <inertial>
-                <mass value="${wheel_weight}"/>
-                <origin xyz="0 0 0" rpy="${pi/2} 0 0"/>
-                <inertia ixx="${(1.0/12.0) * wheel_weight * (3*wheel_radius*wheel_radius + wheel_width*wheel_width)}" ixy="0" ixz="0"
-                         iyy="${(1.0/12.0) * wheel_weight * (3*wheel_radius*wheel_radius + wheel_width*wheel_width)}" iyz="0"
-                         izz="${(1.0/2.0)  * wheel_weight * wheel_radius*wheel_radius}"/>
-            </inertial>
-        </link>
-        <joint name="${name}_joint" type="continuous">
-            <parent link="${parent}"/>
-            <child link="${name}_link"/>
-            <origin xyz="${x} ${y} ${height_offset}" rpy="0 0 0"/>
-            <axis xyz="0 1 0"/>
-            <!-- Damping (Н·м·с/рад): создаёт сопротивление, пропорциональное скорости.
-            Это предотвратит «бесконечное» вращение колес по инерции.-->
-            <!-- Friction (Н·м): минимальное усилие, нужное для начала вращения.
-            Помогает робоу удерживаться на месте и не «дрейфовать» от вибраций.-->
-            <limit effort="1000.0" velocity="20.0"/>
-            <dynamics damping="1.5" friction="1.0"/>
-        </joint>
-        <gazebo reference="${name}_link">
-            <visual>
-                <material>
-                    <ambient>0.1 0.1 0.1 1.0</ambient>
-                    <diffuse>0.1 0.1 0.1 1.0</diffuse>
-                    <specular>0.5 0.5 0.5 1.0</specular>
-                </material>
-            </visual>
-            <collision>
-                <surface>
-                    <friction>
-                        <ode>
-                            <fdir1 ignition:expressed_in="base_footprint">${fdir}</fdir1>   <!-- Ось роликов        -->
-                            <mu>0.05</mu>   <!-- Коэффициент трения вдоль оси fdir  (должен быть 0, чтобы катилось).-->
-                            <mu2>1.0</mu2>  <!-- Коэффициент трения поперёк оси fdir(должен быть 1, чтобы катилось).-->
-                        </ode>
-                    </friction>
-                    <contact>
-                        <ode>
-                            <kp>1e8</kp>
-                            <kd>10.0</kd>
-                            <min_depth>0.001</min_depth>
-                        </ode>
-                    </contact>
-                </surface>
-            </collision>
-        </gazebo>
-    </xacro:macro>
+<!-- Copyright 2026 vladubase                                         -->
+<!--                                                                  -->
+<!-- Licensed under the Apache License, Version 2.0 (the "License");  -->
+<!-- you may not use this file except in compliance with the License. -->
+  <xacro:property name="wheel_radius" value="0.127"/>
+  <xacro:property name="wheel_width"  value="0.132"/>
+  <xacro:property name="wheel_weight" value="10.0"/>
+  <xacro:macro name="mecanum_wheel" params="name x y sx sy parent height_offset fdir">
+    <link name="${name}_link">
+      <visual>
+        <origin xyz="0 0 0" rpy="${pi/2} 0 0"/>
+        <geometry>
+          <mesh filename="package://mona_description/meshes/wheels/mecanum_wheel.stl" scale="${0.001 * sx} ${0.001 * sy} 0.001"/>
+        </geometry>
+        <material name="black">
+          <color rgba="0.1 0.1 0.1 1.0"/>
+        </material>
+      </visual>
+      <collision>
+        <origin xyz="0 0 0" rpy="${pi/2} 0 0"/>
+        <geometry>
+          <sphere radius="${wheel_radius}"/>
+        </geometry>
+      </collision>
+      <inertial>
+        <mass value="${wheel_weight}"/>
+        <origin xyz="0 0 0" rpy="${pi/2} 0 0"/>
+        <inertia ixx="${(1.0/12.0) * wheel_weight * (3*wheel_radius*wheel_radius + wheel_width*wheel_width)}" ixy="0" ixz="0" iyy="${(1.0/12.0) * wheel_weight * (3*wheel_radius*wheel_radius + wheel_width*wheel_width)}" iyz="0" izz="${(1.0/2.0) * wheel_weight * wheel_radius*wheel_radius}"/>
+      </inertial>
+    </link>
+    <joint name="${name}_joint" type="continuous">
+      <parent link="${parent}"/>
+      <child link="${name}_link"/>
+      <origin xyz="${x} ${y} ${height_offset}" rpy="0 0 0"/>
+      <axis xyz="0 1 0"/>
+      <!-- Damping (Н·м·с/рад): создаёт сопротивление, пропорциональное скорости. Это предотвратит «бесконечное» вращение колес по инерции.-->
+      <!-- Friction (Н·м): минимальное усилие, нужное для начала вращения. Помогает робоу удерживаться на месте и не «дрейфовать» от вибраций.-->
+      <limit effort="1000.0" velocity="20.0"/>
+      <dynamics damping="1.5" friction="1.0"/>
+    </joint>
+    <gazebo reference="${name}_link">
+      <visual>
+        <material>
+          <ambient>0.1 0.1 0.1 1.0</ambient>
+          <diffuse>0.1 0.1 0.1 1.0</diffuse>
+          <specular>0.5 0.5 0.5 1.0</specular>
+        </material>
+      </visual>
+      <collision>
+        <surface>
+          <friction>
+            <ode>
+              <fdir1 ignition:expressed_in="base_footprint">${fdir}</fdir1>           <!-- Ось роликов -->
+              <mu>0.05</mu>   <!-- Коэффициент трения вдоль оси fdir (должен быть 0, чтобы катилось).  -->
+              <mu2>1.0</mu2>  <!-- Коэффициент трения поперёк оси fdir(должен быть 1, чтобы катилось). -->
+            </ode>
+          </friction>
+          <contact>
+            <ode>
+              <kp>1e8</kp>
+              <kd>10.0</kd>
+              <min_depth>0.001</min_depth>
+            </ode>
+          </contact>
+        </surface>
+      </collision>
+    </gazebo>
+  </xacro:macro>
 </robot>
