Commit message: feat: add optimized base mesh and IMU sensor

File: src/mona_description/urdf/lidar.xacro (robot description, xacro)
@@ -1,8 +1,8 @@
 <?xml version="1.0"?>
 <robot xmlns:xacro="http://www.ros.org/wiki/xacro">
+    <xacro:property name="lidar_radius" value="0.055"/>
+    <xacro:property name="lidar_height" value="0.080"/>
+    <xacro:property name="lidar_weight" value="0.070"/>
     <xacro:macro name="lidar_sensor" params="name parent *origin">
-        <xacro:property name="lidar_radius" value="0.055"/>
-        <xacro:property name="lidar_height" value="0.080"/>
-        <xacro:property name="lidar_weight" value="0.070"/>
         <joint name="${name}_joint" type="fixed">
             <xacro:insert_block name="origin" />
@@ -33,8 +33,8 @@
                     <scan>
                         <horizontal>
-                            <samples>100</samples>
+                            <samples>300</samples>
                             <resolution>1</resolution>
-                            <min_angle>${-pi/3.6}</min_angle>
-                            <max_angle>${pi/3.6}</max_angle>
+                            <min_angle>${-pi/2.4}</min_angle>
+                            <max_angle>${pi/2.4}</max_angle>
                         </horizontal>
                     </scan>

File: src/mona_description/urdf/mona.urdf.xacro (robot description, xacro)
@@ -3,4 +3,5 @@
     <xacro:include filename="wheel.xacro"/>
     <xacro:include filename="lidar.xacro"/>
+    <xacro:include filename="imu.xacro"/>
     <material name="orange">
         <color rgba="1.0 0.5 0.0 1.0"/>
@@ -12,13 +13,13 @@
     <xacro:property name="robot_road_clearance" value="0.02"/>
     <xacro:property name="wheel_base_x" value="${0.8 / 2}"/>
-    <xacro:property name="wheel_base_y" value="${base_width/2 + wheel_width/2 + 0.002}"/>
+    <xacro:property name="wheel_base_y" value="${base_width/2   - wheel_width/2}"/>
     <xacro:property name="wheel_base_z" value="${-base_height/2 - robot_road_clearance + wheel_radius}"/>
-    <xacro:property name="lidar_offset_x" value="0.58"/>
-    <xacro:property name="lidar_offset_y" value="0.36"/>
-    <xacro:property name="lidar_offset_z" value="-0.05"/>
+    <xacro:property name="lidar_offset_x" value="${base_length/2 - 0.06}"/>
+    <xacro:property name="lidar_offset_y" value="${base_width/2  - 0.06}"/>
+    <xacro:property name="lidar_offset_z" value="${-lidar_height/2}"/>
     <xacro:property name="robot_spawn_x" value="0.0"/>
     <xacro:property name="robot_spawn_y" value="0.0"/>
     <xacro:property name="robot_spawn_z" value="${(robot_road_clearance+0.003) + (base_height/2)}"/>
-    <xacro:property name="lidar_cutout_gap" value="0.15"/>
+    <xacro:property name="lidar_cutout_gap" value="0.50"/>
     <xacro:property name="cap_thickness"    value="0.02"/>
     <xacro:property name="quad_len" value="${(base_length - lidar_cutout_gap)/2}"/>
@@ -34,80 +35,16 @@
     </joint>
     <link name="base_link">
+    <!-- ROBOT BASE -->
         <visual>
-            <origin xyz="0 0 ${base_height/2 - cap_thickness/2}" rpy="0 0 0"/>
+            <origin xyz="0 0 0" rpy="0 0 0"/>
             <geometry>
-                <box size="${base_length} ${base_width} ${cap_thickness}"/>
-            </geometry>
-            <material name="orange"/>
-        </visual>
-        <visual>
-            <origin xyz="0 0 ${-base_height/2 + cap_thickness/2}" rpy="0 0 0"/>
-            <geometry>
-                <box size="${base_length} ${base_width} ${cap_thickness}"/>
-            </geometry>
-            <material name="orange"/>
-        </visual>
-        <visual>
-            <origin xyz="${quad_x_off} ${quad_y_off} 0" rpy="0 0 0"/>
-            <geometry>
-                <box size="${quad_len} ${quad_wid} ${quad_h}"/>
-            </geometry>
-            <material name="orange"/>
-        </visual>
-        <visual>
-            <origin xyz="${quad_x_off} -${quad_y_off} 0" rpy="0 0 0"/>
-            <geometry>
-                <box size="${quad_len} ${quad_wid} ${quad_h}"/>
-            </geometry>
-            <material name="orange"/>
-        </visual>
-        <visual>
-            <origin xyz="-${quad_x_off} ${quad_y_off} 0" rpy="0 0 0"/>
-            <geometry>
-                <box size="${quad_len} ${quad_wid} ${quad_h}"/>
-            </geometry>
-            <material name="orange"/>
-        </visual>
-        <visual>
-            <origin xyz="-${quad_x_off} -${quad_y_off} 0" rpy="0 0 0"/>
-            <geometry>
-                <box size="${quad_len} ${quad_wid} ${quad_h}"/>
+                <mesh filename="package://mona_description/meshes/base.stl" scale="0.001 0.001 0.001"/>
             </geometry>
             <material name="orange"/>
         </visual>
         <collision>
-            <origin xyz="0 0 ${base_height/2 - cap_thickness/2}" rpy="0 0 0"/>
+            <origin xyz="0 0 0" rpy="0 0 0"/>
             <geometry>
-                <box size="${base_length} ${base_width} ${cap_thickness}"/>
-            </geometry>
-        </collision>
-        <collision>
-            <origin xyz="0 0 ${-base_height/2 + cap_thickness/2}" rpy="0 0 0"/>
-            <geometry>
-                <box size="${base_length} ${base_width} ${cap_thickness}"/>
-            </geometry>
-        </collision>
-        <collision>
-            <origin xyz="${quad_x_off} ${quad_y_off} 0" rpy="0 0 0"/>
-            <geometry>
-                <box size="${quad_len} ${quad_wid} ${quad_h}"/>
-            </geometry>
-        </collision>
-        <collision>
-            <origin xyz="${quad_x_off} -${quad_y_off} 0" rpy="0 0 0"/>
-            <geometry>
-                <box size="${quad_len} ${quad_wid} ${quad_h}"/>
-            </geometry>
-        </collision>
-        <collision>
-            <origin xyz="-${quad_x_off} ${quad_y_off} 0" rpy="0 0 0"/>
-            <geometry>
-                <box size="${quad_len} ${quad_wid} ${quad_h}"/>
-            </geometry>
-        </collision>
-        <collision>
-            <origin xyz="-${quad_x_off} -${quad_y_off} 0" rpy="0 0 0"/>
-            <geometry>
-                <box size="${quad_len} ${quad_wid} ${quad_h}"/>
+                <mesh filename="package://mona_description/meshes/base.stl" scale="0.001 0.001 0.001"/>
             </geometry>
         </collision>
@@ -122,8 +59,10 @@
         <material>Gazebo/Orange</material>
     </gazebo>
+    <!-- WHEELS -->
     <xacro:mecanum_wheel name="wheel_front_left"  x="${wheel_base_x}"  y="${wheel_base_y}"  flip_visual="1"  parent="base_link" height_offset="${wheel_base_z}"/>
     <xacro:mecanum_wheel name="wheel_rear_left"   x="-${wheel_base_x}" y="${wheel_base_y}"  flip_visual="1"  parent="base_link" height_offset="${wheel_base_z}"/>
     <xacro:mecanum_wheel name="wheel_front_right" x="${wheel_base_x}"  y="-${wheel_base_y}" flip_visual="-1" parent="base_link" height_offset="${wheel_base_z}"/>
     <xacro:mecanum_wheel name="wheel_rear_right"  x="-${wheel_base_x}" y="-${wheel_base_y}" flip_visual="-1" parent="base_link" height_offset="${wheel_base_z}"/>
+    <!-- LIDARS -->
     <xacro:lidar_sensor name="lidar_front" parent="base_link">
         <origin xyz="${lidar_offset_x} 0 ${lidar_offset_z}" rpy="0 0 0"/>
@@ -138,4 +77,8 @@
         <origin xyz="0 -${lidar_offset_y} ${lidar_offset_z}" rpy="0 0 -${pi/2}"/>
     </xacro:lidar_sensor>
+    <!-- IMU -->
+    <xacro:imu_sensor name="imu" parent="base_link">
+        <origin xyz="0 0 0" rpy="0 0 0"/>
+    </xacro:imu_sensor>
     <gazebo>
         <plugin name="object_controller" filename="libgazebo_ros_planar_move.so">
@@ -151,4 +94,14 @@
             <publish_odom_tf>true</publish_odom_tf>
         </plugin>
+        <plugin name="joint_state_publisher" filename="libgazebo_ros_joint_state_publisher.so">
+            <ros>
+                <remapping>~/out:=joint_states</remapping>
+            </ros>
+            <update_rate>30</update_rate>
+            <joint_name>wheel_front_left_joint</joint_name>
+            <joint_name>wheel_front_right_joint</joint_name>
+            <joint_name>wheel_rear_left_joint</joint_name>
+            <joint_name>wheel_rear_right_joint</joint_name>
+        </plugin>
     </gazebo>
 </robot>

File: src/mona_description/urdf/wheel.xacro (robot description, xacro)
@@ -2,5 +2,5 @@
 <robot xmlns:xacro="http://www.ros.org/wiki/xacro">
     <xacro:property name="wheel_radius" value="0.127"/>
-    <xacro:property name="wheel_width"  value="0.10"/>
+    <xacro:property name="wheel_width"  value="0.132"/>
     <xacro:property name="wheel_weight" value="15.0"/>
     <xacro:macro name="mecanum_wheel" params="name x y flip_visual parent height_offset">
@@ -9,5 +9,5 @@
                 <origin xyz="0 0 0" rpy="${pi/2} 0 0"/>
                 <geometry>
-                    <cylinder radius="${wheel_radius}" length="${wheel_width}"/>
+                    <mesh filename="package://mona_description/meshes/wheels/mecanum_wheel.stl" scale="0.001 0.001 0.001"/>
                 </geometry>
                 <material name="black">
@@ -26,5 +26,5 @@
                 <inertia ixx="${(1.0/12.0) * wheel_weight * (3*wheel_radius*wheel_radius + wheel_width*wheel_width)}" ixy="0" ixz="0"
                          iyy="${(1.0/12.0) * wheel_weight * (3*wheel_radius*wheel_radius + wheel_width*wheel_width)}" iyz="0"
-                         izz="${(1.0/2.0) * wheel_weight * wheel_radius*wheel_radius}"/>
+                         izz="${(1.0/2.0)  * wheel_weight * wheel_radius*wheel_radius}"/>
             </inertial>
         </link>

Commit message: Refactor: Integrate safety logic into mona_core.
- Moved safety_node and bringup launch to mona_core package.
- Removed deprecated mona_safety package.
- Updated linter configurations (uncrustify/setup.cfg) for strict formatting.
- Implemented watchdog timer and guard clauses in SafetyNode.
- Enforced strict clean build policy in run scripts.

File: src/mona_description/urdf/lidar.xacro (robot description, xacro)
@@ -14,7 +14,14 @@
   <!-- See the License for the specific language governing permissions and      -->
   <!-- limitations under the License.                                           -->
-  <xacro:property name="lidar_radius" value="0.055"/>
-  <xacro:property name="lidar_height" value="0.080"/>
-  <xacro:property name="lidar_weight" value="0.070"/>
+  <!--           SLAMTEC              -->
+  <!--      LPX-E3 Series E3P2        -->
+  <!-- https://www.slamtec.com/en/E3  -->
+  <xacro:property name="lidar_radius"     value="0.057"/>
+  <xacro:property name="lidar_height"     value="0.048"/>
+  <xacro:property name="lidar_weight"     value="0.180"/>
+  <xacro:property name="lidar_fov"        value="150"/>
+  <xacro:property name="lidar_res_angle"  value="0.17"/>
+  <xacro:property name="lidar_samples"    value="${lidar_fov / lidar_res_angle}"/>
+  <xacro:property name="lidar_updaterate" value="15"/>
   <xacro:macro name="lidar_sensor" params="name parent *origin">
     <link name="${name}_link">
@@ -43,5 +50,5 @@
         <always_on>true</always_on>
         <visualize>true</visualize>
-        <update_rate>10</update_rate>
+        <update_rate>${lidar_updaterate}</update_rate>
         <gz_frame_id>${name}_link</gz_frame_id>
         <ign_frame_id>${name}_link</ign_frame_id>
@@ -49,5 +56,5 @@
           <scan>
             <horizontal>
-              <samples>300</samples>
+              <samples>${lidar_samples}</samples>
               <resolution>1</resolution>
               <min_angle>${-pi/2.4}</min_angle>
@@ -57,11 +64,11 @@
           <range>
             <min>0.10</min>
-            <max>20.0</max>
-            <resolution>0.01</resolution>
+            <max>40.0</max>
+            <resolution>0.1</resolution>
           </range>
           <noise>
             <type>gaussian</type>
             <mean>0.0</mean>
-            <stddev>0.01</stddev>
+            <stddev>0.03</stddev>
           </noise>
         </ray>
