Commit message: feat: added working LiDAR configuration and fixed collision issues

File: src/mona_description/urdf/mona.urdf.xacro (robot description, xacro)
@@ -1,18 +1,30 @@
 <?xml version="1.0"?>
 <robot xmlns:xacro="http://www.ros.org/wiki/xacro" name="mona">
+    <xacro:include filename="wheel.xacro"/>
+    <xacro:include filename="lidar.xacro"/>
+    <material name="orange">
+        <color rgba="1.0 0.5 0.0 1.0"/>
+    </material>
     <xacro:property name="base_length"  value="1.25"/>
     <xacro:property name="base_width"   value="0.80"/>
     <xacro:property name="base_height"  value="0.30"/>
-    <xacro:property name="base_mass"    value="150.0"/>
+    <xacro:property name="base_weight"  value="150.0"/>
     <xacro:property name="robot_road_clearance" value="0.02"/>
-    <xacro:property name="wheel_radius" value="0.127"/>
-    <xacro:property name="wheel_width"  value="0.10"/>
-    <xacro:property name="wheel_mass"   value="15.0"/>
     <xacro:property name="wheel_base_x" value="${0.8 / 2}"/>
     <xacro:property name="wheel_base_y" value="${base_width/2 + wheel_width/2 + 0.002}"/>
     <xacro:property name="wheel_base_z" value="${-base_height/2 - robot_road_clearance + wheel_radius}"/>
+    <xacro:property name="lidar_offset_x" value="0.58"/>
+    <xacro:property name="lidar_offset_y" value="0.36"/>
+    <xacro:property name="lidar_offset_z" value="-0.05"/>
     <xacro:property name="robot_spawn_x" value="0.0"/>
     <xacro:property name="robot_spawn_y" value="0.0"/>
     <xacro:property name="robot_spawn_z" value="${(robot_road_clearance+0.003) + (base_height/2)}"/>
+    <xacro:property name="lidar_cutout_gap" value="0.15"/>
+    <xacro:property name="cap_thickness"    value="0.02"/>
+    <xacro:property name="quad_len" value="${(base_length - lidar_cutout_gap)/2}"/>
+    <xacro:property name="quad_wid" value="${(base_width - lidar_cutout_gap)/2}"/>
+    <xacro:property name="quad_h"   value="${base_height - 2*cap_thickness}"/>
+    <xacro:property name="quad_x_off" value="${(lidar_cutout_gap + quad_len)/2}"/>
+    <xacro:property name="quad_y_off" value="${(lidar_cutout_gap + quad_wid)/2}"/>
     <link name="base_footprint"/>
     <joint name="base_joint" type="fixed">
@@ -23,21 +35,86 @@
     <link name="base_link">
         <visual>
+            <origin xyz="0 0 ${base_height/2 - cap_thickness/2}" rpy="0 0 0"/>
             <geometry>
-                <box size="${base_length} ${base_width} ${base_height}"/>
+                <box size="${base_length} ${base_width} ${cap_thickness}"/>
             </geometry>
-            <material name="orange">
-                <color rgba="1.0 0.5 0.0 1.0"/>
-            </material>
+            <material name="orange"/>
+        </visual>
+        <visual>
+            <origin xyz="0 0 ${-base_height/2 + cap_thickness/2}" rpy="0 0 0"/>
+            <geometry>
+                <box size="${base_length} ${base_width} ${cap_thickness}"/>
+            </geometry>
+            <material name="orange"/>
+        </visual>
+        <visual>
+            <origin xyz="${quad_x_off} ${quad_y_off} 0" rpy="0 0 0"/>
+            <geometry>
+                <box size="${quad_len} ${quad_wid} ${quad_h}"/>
+            </geometry>
+            <material name="orange"/>
+        </visual>
+        <visual>
+            <origin xyz="${quad_x_off} -${quad_y_off} 0" rpy="0 0 0"/>
+            <geometry>
+                <box size="${quad_len} ${quad_wid} ${quad_h}"/>
+            </geometry>
+            <material name="orange"/>
+        </visual>
+        <visual>
+            <origin xyz="-${quad_x_off} ${quad_y_off} 0" rpy="0 0 0"/>
+            <geometry>
+                <box size="${quad_len} ${quad_wid} ${quad_h}"/>
+            </geometry>
+            <material name="orange"/>
+        </visual>
+        <visual>
+            <origin xyz="-${quad_x_off} -${quad_y_off} 0" rpy="0 0 0"/>
+            <geometry>
+                <box size="${quad_len} ${quad_wid} ${quad_h}"/>
+            </geometry>
+            <material name="orange"/>
         </visual>
         <collision>
+            <origin xyz="0 0 ${base_height/2 - cap_thickness/2}" rpy="0 0 0"/>
             <geometry>
-                <box size="${base_length} ${base_width} ${base_height}"/>
+                <box size="${base_length} ${base_width} ${cap_thickness}"/>
+            </geometry>
+        </collision>
+        <collision>
+            <origin xyz="0 0 ${-base_height/2 + cap_thickness/2}" rpy="0 0 0"/>
+            <geometry>
+                <box size="${base_length} ${base_width} ${cap_thickness}"/>
+            </geometry>
+        </collision>
+        <collision>
+            <origin xyz="${quad_x_off} ${quad_y_off} 0" rpy="0 0 0"/>
+            <geometry>
+                <box size="${quad_len} ${quad_wid} ${quad_h}"/>
+            </geometry>
+        </collision>
+        <collision>
+            <origin xyz="${quad_x_off} -${quad_y_off} 0" rpy="0 0 0"/>
+            <geometry>
+                <box size="${quad_len} ${quad_wid} ${quad_h}"/>
+            </geometry>
+        </collision>
+        <collision>
+            <origin xyz="-${quad_x_off} ${quad_y_off} 0" rpy="0 0 0"/>
+            <geometry>
+                <box size="${quad_len} ${quad_wid} ${quad_h}"/>
+            </geometry>
+        </collision>
+        <collision>
+            <origin xyz="-${quad_x_off} -${quad_y_off} 0" rpy="0 0 0"/>
+            <geometry>
+                <box size="${quad_len} ${quad_wid} ${quad_h}"/>
             </geometry>
         </collision>
         <inertial>
-            <mass value="${base_mass}"/>
-            <inertia ixx="${(1/12) * base_mass * (base_width * base_width + base_height*base_height)}" ixy="0.0" ixz="0.0"
-                     iyy="${(1/12) * base_mass * (base_length*base_length + base_height*base_height)}" iyz="0.0"
-                     izz="${(1/12) * base_mass * (base_length*base_length + base_width*base_width)}"/>
+            <mass value="${base_weight}"/>
+            <inertia ixx="${(1.0/12.0) * base_weight * (base_width * base_width + base_height*base_height)}" ixy="0.0" ixz="0.0"
+                     iyy="${(1.0/12.0) * base_weight * (base_length*base_length + base_height*base_height)}" iyz="0.0"
+                     izz="${(1.0/12.0) * base_weight * (base_length*base_length + base_width*base_width)}"/>
         </inertial>
     </link>
@@ -45,44 +122,20 @@
         <material>Gazebo/Orange</material>
     </gazebo>
-    <xacro:macro name="mecanum_wheel" params="name x y flip_visual">
-        <link name="${name}_link">
-            <visual>
-                <origin xyz="0 0 0" rpy="${pi/2} 0 0"/> <geometry>
-                    <cylinder radius="${wheel_radius}" length="${wheel_width}"/>
-                    </geometry>
-                <material name="black">
-                    <color rgba="0.1 0.1 0.1 1.0"/>
-                </material>
-            </visual>
-            <collision>
-                <origin xyz="0 0 0" rpy="${pi/2} 0 0"/>
-                <geometry>
-                    <cylinder radius="${wheel_radius}" length="${wheel_width}"/>
-                </geometry>
-            </collision>
-            <inertial>
-                <mass value="${wheel_mass}"/>
-                <origin xyz="0 0 0" rpy="${pi/2} 0 0"/>
-                <inertia ixx="${(1/12) * wheel_mass * (3*wheel_radius*wheel_radius + wheel_width*wheel_width)}" ixy="0" ixz="0"
-                         iyy="${(1/12) * wheel_mass * (3*wheel_radius*wheel_radius + wheel_width*wheel_width)}" iyz="0"
-                         izz="${(1/2) * wheel_mass * wheel_radius*wheel_radius}"/>
-            </inertial>
-        </link>
-        <joint name="${name}_joint" type="continuous">
-            <parent link="base_link"/>
-            <child link="${name}_link"/>
-            <origin xyz="${x} ${y} ${wheel_base_z}" rpy="0 0 0"/>
-            <axis xyz="0 1 0"/>
-        </joint>
-        <gazebo reference="${name}_link">
-            <material>Gazebo/Grey</material>
-            <mu1>0.8</mu1>
-            <mu2>0.8</mu2>
-        </gazebo>
-    </xacro:macro>
-    <xacro:mecanum_wheel name="wheel_front_left"  x="${wheel_base_x}"  y="${wheel_base_y}"  flip_visual="1"/>
-    <xacro:mecanum_wheel name="wheel_rear_left"   x="-${wheel_base_x}" y="${wheel_base_y}"  flip_visual="1"/>
-    <xacro:mecanum_wheel name="wheel_front_right" x="${wheel_base_x}"  y="-${wheel_base_y}" flip_visual="-1"/>
-    <xacro:mecanum_wheel name="wheel_rear_right"  x="-${wheel_base_x}" y="-${wheel_base_y}" flip_visual="-1"/>
+    <xacro:mecanum_wheel name="wheel_front_left"  x="${wheel_base_x}"  y="${wheel_base_y}"  flip_visual="1"  parent="base_link" height_offset="${wheel_base_z}"/>
+    <xacro:mecanum_wheel name="wheel_rear_left"   x="-${wheel_base_x}" y="${wheel_base_y}"  flip_visual="1"  parent="base_link" height_offset="${wheel_base_z}"/>
+    <xacro:mecanum_wheel name="wheel_front_right" x="${wheel_base_x}"  y="-${wheel_base_y}" flip_visual="-1" parent="base_link" height_offset="${wheel_base_z}"/>
+    <xacro:mecanum_wheel name="wheel_rear_right"  x="-${wheel_base_x}" y="-${wheel_base_y}" flip_visual="-1" parent="base_link" height_offset="${wheel_base_z}"/>
+    <xacro:lidar_sensor name="lidar_front" parent="base_link">
+        <origin xyz="${lidar_offset_x} 0 ${lidar_offset_z}" rpy="0 0 0"/>
+    </xacro:lidar_sensor>
+    <xacro:lidar_sensor name="lidar_rear" parent="base_link">
+        <origin xyz="-${lidar_offset_x} 0 ${lidar_offset_z}" rpy="0 0 ${pi}"/>
+    </xacro:lidar_sensor>
+    <xacro:lidar_sensor name="lidar_left" parent="base_link">
+        <origin xyz="0 ${lidar_offset_y} ${lidar_offset_z}" rpy="0 0 ${pi/2}"/>
+    </xacro:lidar_sensor>
+    <xacro:lidar_sensor name="lidar_right" parent="base_link">
+        <origin xyz="0 -${lidar_offset_y} ${lidar_offset_z}" rpy="0 0 -${pi/2}"/>
+    </xacro:lidar_sensor>
     <gazebo>
         <plugin name="object_controller" filename="libgazebo_ros_planar_move.so">

Commit message: feat: add static LED mesh and optimize docker/launch config

File: src/mona_description/urdf/mona.urdf.xacro (robot description, xacro)
@@ -21,11 +21,5 @@
     <xacro:property name="robot_spawn_y" value="0.0"/>
     <xacro:property name="robot_spawn_z" value="${(robot_road_clearance+0.003) + (base_height/2)}"/>
-    <xacro:property name="lidar_cutout_gap" value="0.50"/>
-    <xacro:property name="cap_thickness"    value="0.02"/>
-    <xacro:property name="quad_len" value="${(base_length - lidar_cutout_gap)/2}"/>
-    <xacro:property name="quad_wid" value="${(base_width - lidar_cutout_gap)/2}"/>
-    <xacro:property name="quad_h"   value="${base_height - 2*cap_thickness}"/>
-    <xacro:property name="quad_x_off" value="${(lidar_cutout_gap + quad_len)/2}"/>
-    <xacro:property name="quad_y_off" value="${(lidar_cutout_gap + quad_wid)/2}"/>
+    <!-- BASE FOOTPRINT -->
     <link name="base_footprint"/>
     <joint name="base_joint" type="fixed">
@@ -34,6 +28,6 @@
         <origin xyz="${robot_spawn_x} ${robot_spawn_y} ${robot_spawn_z}" rpy="0 0 0"/>
     </joint>
+    <!-- ROBOT BASE -->
     <link name="base_link">
-    <!-- ROBOT BASE -->
         <visual>
             <origin xyz="0 0 0" rpy="0 0 0"/>
@@ -81,8 +75,29 @@
         <origin xyz="0 0 0" rpy="0 0 0"/>
     </xacro:imu_sensor>
+    <!-- LED -->
+    <link name="led_strip_link">
+        <visual>
+            <origin xyz="0 0 0" rpy="0 0 0"/>
+            <geometry>
+                <mesh filename="package://mona_description/meshes/led.stl" scale="0.001 0.001 0.001"/>
+            </geometry>
+            <material name="white">
+                <color rgba="1.0 1.0 1.0 0.8"/>
+            </material>
+        </visual>
+    </link>
+    <joint name="led_strip_joint" type="fixed">
+        <parent link="base_link"/>
+        <child link="led_strip_link"/>
+        <origin xyz="0 0 ${base_height/2 - 0.025}" rpy="0 0 0"/>
+    </joint>
+    <gazebo reference="led_strip_link">
+        <material>Gazebo/WhiteGlow</material>
+    </gazebo>
+    <!-- PLUGIN CONNECTIONS -->
     <gazebo>
         <plugin name="object_controller" filename="libgazebo_ros_planar_move.so">
             <ros>
-                <argument>odom:=odom/unfiltered</argument>
+                <remapping>odom:=odom/unfiltered</remapping>
             </ros>
             <command_topic>cmd_vel</command_topic>

Commit message: feat: add front camera URDF and gazebo bridge

File: src/mona_description/urdf/mona.urdf.xacro (robot description, xacro)
@@ -19,4 +19,5 @@
   <xacro:include filename="lidar.xacro"/>
   <xacro:include filename="imu.xacro"/>
+  <xacro:include filename="camera.xacro"/>
   <material name="orange">
     <color rgba="1.0 0.5 0.0 1.0"/>
@@ -89,4 +90,8 @@
     <origin xyz="0 0 0" rpy="0 0 0"/>
   </xacro:imu_sensor>
+  <!-- CAMERA -->
+  <xacro:camera_sensor name="camera" parent="base_link">
+    <origin xyz="${base_length/2} 0 -0.065" rpy="0 0 0"/>
+  </xacro:camera_sensor>
   <!-- LED -->
   <link name="led_strip_link">

File: src/mona_description/urdf/wheel.xacro (robot description, xacro)
@@ -2,8 +2,17 @@
 <robot xmlns:xacro="http://www.ros.org/wiki/xacro"
        xmlns:ignition="http://gazebosim.org/schema">
-<!-- Copyright 2026 vladubase                                         -->
-<!--                                                                  -->
-<!-- Licensed under the Apache License, Version 2.0 (the "License");  -->
-<!-- you may not use this file except in compliance with the License. -->
+  <!-- Copyright 2026 vladubase                                                 -->
+  <!--                                                                          -->
+  <!-- Licensed under the Apache License, Version 2.0 (the "License");          -->
+  <!-- you may not use this file except in compliance with the License.         -->
+  <!-- You may obtain a copy of the License at                                  -->
+  <!--                                                                          -->
+  <!-- http://www.apache.org/licenses/LICENSE-2.0                               -->
+  <!--                                                                          -->
+  <!-- Unless required by applicable law or agreed to in writing, software      -->
+  <!-- distributed under the License is distributed on an "AS IS" BASIS,        -->
+  <!-- WITHOUT WARRANTIES OR CONDITIONS OF ANY KIND, either express or implied. -->
+  <!-- See the License for the specific language governing permissions and      -->
+  <!-- limitations under the License.                                           -->
   <xacro:property name="wheel_radius" value="0.127"/>
   <xacro:property name="wheel_width"  value="0.132"/>
