Commit message: feat(core): introduce FDIR manager, swarm namespaces and dynamic URDF
- Add Python FDIR Lifecycle Manager
- Refactor launch files (robot.launch, world.launch) for Swarm scaling
- Update Foxglove dashboard layout and configs
- Adapt URDF/Xacro for dynamic tf_prefix/namespace injection

File: src/mona_description/urdf/camera.xacro (robot description, xacro)
@@ -50,6 +50,7 @@
         <update_rate>30.0</update_rate>
         <visualize>true</visualize>
-        <topic>/camera/image_raw</topic>
-        <ignition_frame_id>${name}_optical_link</ignition_frame_id>
+        <topic>/$(arg namespace)/camera/image_raw</topic>
+        <ignition_frame_id>$(arg namespace)/${name}_optical_link</ignition_frame_id>
+        <gz_frame_id>$(arg namespace)/${name}_optical_link</gz_frame_id>
         <camera>
           <horizontal_fov>1.3962634</horizontal_fov>

File: src/mona_description/urdf/imu.xacro (robot description, xacro)
@@ -40,7 +40,8 @@
         <update_rate>100</update_rate>
         <visualize>false</visualize>
-        <topic>/${name}/data</topic>
+        <topic>/$(arg namespace)/${name}/data</topic>
         <pose>0 0 0 0 0 0</pose>
-        <ignition_frame_id>${name}_link</ignition_frame_id>
+        <ignition_frame_id>$(arg namespace)/${name}_link</ignition_frame_id>
+        <gz_frame_id>$(arg namespace)/${name}_link</gz_frame_id>
         <imu>
           <angular_velocity>

File: src/mona_description/urdf/lidar.xacro (robot description, xacro)
@@ -45,12 +45,13 @@
     </joint>
     <gazebo reference="${name}_link">
-      <sensor name="${name}" type="gpu_lidar">  <!-- or 'lidar' -->
+      <sensor name="${name}" type="gpu_lidar">
         <pose>0 0 0 0 0 0</pose>
-        <topic>${name}/scan</topic>
+        <topic>/$(arg namespace)/${name}/scan</topic>
         <always_on>true</always_on>
         <visualize>true</visualize>
         <update_rate>${lidar_updaterate}</update_rate>
-        <gz_frame_id>${name}_link</gz_frame_id>
-        <ign_frame_id>${name}_link</ign_frame_id>
+        <ignition_frame_id>$(arg namespace)/${name}_link</ignition_frame_id>
+        <gz_frame_id>$(arg namespace)/${name}_link</gz_frame_id>
+        <ign_frame_id>$(arg namespace)/${name}_link</ign_frame_id>
         <ray>
           <scan>

File: src/mona_description/urdf/mona.urdf.xacro (robot description, xacro)
@@ -20,4 +20,5 @@
   <xacro:include filename="imu.xacro"/>
   <xacro:include filename="camera.xacro"/>
+  <xacro:arg name="namespace" default=""/>
   <material name="orange">
     <color rgba="1.0 0.5 0.0 1.0"/>
@@ -59,4 +60,5 @@
       <origin xyz="0 0 0" rpy="0 0 0"/>
       <geometry>
+        <!-- <box size="${base_length} ${base_width} ${base_height}"/> -->
         <mesh filename="package://mona_description/meshes/base.stl" scale="0.001 0.001 0.001"/>
       </geometry>
@@ -125,5 +127,5 @@
     <!-- TF -->
     <plugin filename="libignition-gazebo-joint-state-publisher-system.so" name="ignition::gazebo::systems::JointStatePublisher">
-      <topic>joint_states</topic>
+      <topic>/$(arg namespace)/joint_states</topic>
     </plugin>
     <!-- Mecanum Wheels -->
@@ -138,11 +140,12 @@
       <min_acceleration>-2.5</min_acceleration>
       <max_acceleration>2.5</max_acceleration>
-      <topic>/hardware/motor_cmd</topic>
+      <topic>/$(arg namespace)/hardware/motor_cmd</topic>
     </plugin>
     <!-- Sensor: Odometry -->
     <plugin filename="libignition-gazebo-odometry-publisher-system.so" name="ignition::gazebo::systems::OdometryPublisher">
-      <odom_frame>odom</odom_frame>
-      <robot_base_frame>base_footprint</robot_base_frame>
-      <odom_topic>/odom</odom_topic>
+      <odom_frame>$(arg namespace)/odom</odom_frame>
+      <robot_base_frame>$(arg namespace)/base_footprint</robot_base_frame>
+      <odom_topic>/$(arg namespace)/odom</odom_topic>
+      <tf_topic>/$(arg namespace)/tf</tf_topic>
       <odom_publish_frequency>50</odom_publish_frequency>
       <dimensions>3</dimensions>

File: src/mona_description/urdf/wheel.xacro (robot description, xacro)
@@ -46,6 +46,6 @@
       <origin xyz="${x} ${y} ${height_offset}" rpy="0 0 0"/>
       <axis xyz="0 1 0"/>
-      <!-- Damping (Н·м·с/рад): создаёт сопротивление, пропорциональное скорости. Это предотвратит «бесконечное» вращение колес по инерции.-->
-      <!-- Friction (Н·м): минимальное усилие, нужное для начала вращения. Помогает робоу удерживаться на месте и не «дрейфовать» от вибраций.-->
+      <!-- Damping (Nm s/rad): Creates resistance proportional to speed. This prevents the wheels from spinning "infinitely" due to inertia.-->
+      <!-- Friction (Nm): The minimum force required to initiate rotation. Helps the robot stay in place and prevent it from "drifting" due to vibrations.-->
       <limit effort="1000.0" velocity="20.0"/>
       <dynamics damping="1.5" friction="1.0"/>
@@ -63,7 +63,7 @@
           <friction>
             <ode>
-              <fdir1 ignition:expressed_in="base_footprint">${fdir}</fdir1>           <!-- Ось роликов -->
-              <mu>0.05</mu>   <!-- Коэффициент трения вдоль оси fdir (должен быть 0, чтобы катилось).  -->
-              <mu2>1.0</mu2>  <!-- Коэффициент трения поперёк оси fdir(должен быть 1, чтобы катилось). -->
+              <fdir1 ignition:expressed_in="base_footprint">${fdir}</fdir1>   <!-- Roller axis -->
+              <mu>0.05</mu>   <!-- The coefficient of friction along the axis fdir (must be 0 for it to roll). -->
+              <mu2>1.0</mu2>  <!-- The coefficient of friction across the axis fdir(must be 1 for it to roll). -->
             </ode>
           </friction>
